File: matrix.sch (KiCad schematic (older format))
At the start: 150 parts, among them K00 KEYSW, K00_1 KEYSW, K00_2 KEYSW, K00_3 KEYSW, K01 KEYSW, K02 KEYSW, K03 KEYSW, K04 KEYSW, K05 KEYSW, K06 KEYSW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

Commit message: Reroute for stabs
Parts:
- D00, D01, D02, D03, D04, D05, D06, D07, D10, D11, D12, D13, D14, D15, D16, D17, D20, D21, D22, D23, D24, D25, D26, D27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: symbol D-RESCUE-alps64 -> D
